File: hw/power_dist.sch (EAGLE design)
At the start: 97 parts, among them J1 JST-ZH6SMT_VERT, J2 JST-PH4SMT_VERT, J3 JST-PH5VERT, P1 XT30P, P2 XT30P, P3 XT30P, P4 XT30P, P5 XT30P, P6 XT30P, P7 XT90PW-M, Q1 PSMN4R8-100BSEJ, Q2 PSMN4R8-100BSEJ, Q3 PSMN4R8-100BSEJ, U1 MAX15062AATA+T, U2 STM32G474CEU6, U3 TPS2490DGSR, U4 TCAN334G, U5 LT1787HVIMS8PBF, U6 STLM20DD9FUDFN-4L_STM-L

Commit message: Add part numbers, rev to 4.3b
Parts:
- C10, C4: value 10uF 50V -> 10uF; HOUSEPART (none) -> 1; MF TDK -> (none); MPN C3216X7R1H106K160AE -> MF-CAP-1206-10uF
- C12: HOUSEPART 1 -> 0; MPN MF-CAP-0603-0.1uF -> GRM188R72A104KA35D
- C13: HOUSEPART 1 -> 0; MPN (none) -> CL10B273KB8NNNC
- C14: MPN MF-CAP-0603-0.1uF -> MF-CAP-0603-0.01uF
- D6: MPN MMSZ5223BT1G -> MMSZ4682T1G
- P7: POPULATE 0 -> 1
- R11, R13: HOUSEPART 1 -> 0; MPN (none) -> RC0603FR-073ML
- R12, R14, R17, R3: HOUSEPART 1 -> 0; MPN (none) -> RC0603FR-07200KL
- R16, R2: MPN (none) -> MF-RES-0603-100K
- R18: value 100k 1% -> 140k 1%; HOUSEPART 1 -> 0; MPN (none) -> RC0603FR-07140KL
- R19: HOUSEPART 1 -> 0; MPN (none) -> RC0603FR-07499KL
- R20, R7: HOUSEPART 1 -> 0; MPN (none) -> RC0603FR-0747KL
- R21: MPN (none) -> RC0603FR-0733KL
- R22: value 200k 1% -> 100k; MPN (none) -> MF-RES-0603-100K
- R24, R26: MPN (none) -> MF-RES-0603-0
- R25: POPULATE (none) -> 0
- R5: MPN (none) -> MF-RES-0603-10
- R6: MPN (none) -> MF-RES-0603-1K
- R8: HOUSEPART 1 -> 0; MPN (none) -> RC0603FR-076K8L
- U3: MPN (none) -> TPS2490DGSR; POPULATE (none) -> 1
- U5: MPN (none) -> LT1787HVIMS8; POPULATE (none) -> 1
Other:
- note added: "If this is revved, put a zener in parallel with R20 so that R20 can be equal to R22."
Changed lines of the file:
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@@
 </part>
 <part name="P7" library="power_dist" deviceset="XT90" device="PW-M">
-<attribute name="POPULATE" value="0"/>
+<attribute name="POPULATE" value="1"/>
 </part>
 <part name="P1" library="precharge" deviceset="XT30" device="P">
@@
 <attribute name="MPN" value="MF-CAP-0603-1uF"/>
 </part>
-<part name="C10" library="mfpassives" deviceset="CAPACITOR_NP" device="_1206" value="10uF 50V">
-<attribute name="MF" value="TDK"/>
-<attribute name="MPN" value="C3216X7R1H106K160AE"/>
+<part name="C10" library="mfpassives" deviceset="CAPACITOR_NP" device="_1206" value="10uF">
+<attribute name="HOUSEPART" value="1"/>
+<attribute name="MF" value=""/>
+<attribute name="MPN" value="MF-CAP-1206-10uF"/>
 </part>
 <part name="J1" library="precharge" deviceset="JST-ZH6" device="SMT_VERT">
@@
 <attribute name="POPULATE" value="1"/>
 </part>
-<part name="C4" library="mfpassives" deviceset="CAPACITOR_NP" device="_1206" value="10uF 50V">
-<attribute name="MF" value="TDK"/>
-<attribute name="MPN" value="C3216X7R1H106K160AE"/>
+<part name="C4" library="mfpassives" deviceset="CAPACITOR_NP" device="_1206" value="10uF">
+<attribute name="HOUSEPART" value="1"/>
+<attribute name="MF" value=""/>
+<attribute name="MPN" value="MF-CAP-1206-10uF"/>
 </part>
 <part name="P+5" library="supply1" library_urn="urn:adsk.eagle:library:371" deviceset="+24V" device=""/>
@@
 <attribute name="POPULATE" value="0"/>
 </part>
-<part name="U5" library="LT1787HVIMS8PBF" deviceset="LT1787HVIMS8PBF" device=""/>
+<part name="U5" library="LT1787HVIMS8PBF" deviceset="LT1787HVIMS8PBF" device="">
+<attribute name="MPN" value="LT1787HVIMS8"/>
+<attribute name="POPULATE" value="1"/>
+</part>
 <part name="GND10" library="supply1" deviceset="GND" device=""/>
 <part name="C17" library="mfpassives" deviceset="CAPACITOR_NP" device="_0603" value="0.1uF">
@@
 <part name="R5" library="mfpassives" deviceset="RESISTOR" device="_0603" value="10">
 <attribute name="HOUSEPART" value="1"/>
+<attribute name="MPN" value="MF-RES-0603-10"/>
 </part>
 <part name="R6" library="mfpassives" deviceset="RESISTOR" device="_0603" value="1k">
 <attribute name="HOUSEPART" value="1"/>
+<attribute name="MPN" value="MF-RES-0603-1K"/>
 </part>
 <part name="C13" library="mfpassives" deviceset="CAPACITOR_NP" device="_0603" value="27nF">
-<attribute name="HOUSEPART" value="1"/>
+<attribute name="HOUSEPART" value="0"/>
+<attribute name="MPN" value="CL10B273KB8NNNC"/>
 </part>
 <part name="GND13" library="supply1" deviceset="GND" device=""/>
 <part name="C14" library="mfpassives" deviceset="CAPACITOR_NP" device="_0603" value="10nF">
 <attribute name="HOUSEPART" value="1"/>
-<attribute name="MPN" value="MF-CAP-0603-0.1uF"/>
+<attribute name="MPN" value="MF-CAP-0603-0.01uF"/>
 </part>
 <part name="GND21" library="supply1" deviceset="GND" device=""/>
 <part name="R11" library="mfpassives" deviceset="RESISTOR" device="_0603" value="3M 1%">
-<attribute name="HOUSEPART" value="1"/>
+<attribute name="HOUSEPART" value="0"/>
+<attribute name="MPN" value="RC0603FR-073ML"/>
 </part>
 <part name="R12" library="mfpassives" deviceset="RESISTOR" device="_0603" value="200k 1%">
-<attribute name="HOUSEPART" value="1"/>
+<attribute name="HOUSEPART" value="0"/>
+<attribute name="MPN" value="RC0603FR-07200KL"/>
 </part>
 <part name="R13" library="mfpassives" deviceset="RESISTOR" device="_0603" value="3M 1%">
-<attribute name="HOUSEPART" value="1"/>
+<attribute name="HOUSEPART" value="0"/>
+<attribute name="MPN" value="RC0603FR-073ML"/>
 </part>
 <part name="R14" library="mfpassives" deviceset="RESISTOR" device="_0603" value="200k 1%">
-<attribute name="HOUSEPART" value="1"/>
+<attribute name="HOUSEPART" value="0"/>
+<attribute name="MPN" value="RC0603FR-07200KL"/>
 </part>
 <part name="GND25" library="supply1" deviceset="GND" device=""/>
@@
 <part name="R2" library="mfpassives" deviceset="RESISTOR" device="_0603" value="100k">
 <attribute name="HOUSEPART" value="1"/>
+<attribute name="MPN" value="MF-RES-0603-100K"/>
 </part>
 <part name="GND8" library="supply1" deviceset="GND" device=""/>
@@
 <attribute name="POPULATE" value="0"/>
 </part>
-<part name="U3" library="TPS2490DGSR" deviceset="TPS2490DGSR" device=""/>
+<part name="U3" library="TPS2490DGSR" deviceset="TPS2490DGSR" device="">
+<attribute name="MPN" value="TPS2490DGSR"/>
+<attribute name="POPULATE" value="1"/>
+</part>
 <part name="R7" library="mfpassives" deviceset="RESISTOR" device="_0603" value="47k 1%">
-<attribute name="HOUSEPART" value="1"/>
+<attribute name="HOUSEPART" value="0"/>
+<attribute name="MPN" value="RC0603FR-0747KL"/>
 </part>
 <part name="R8" library="mfpassives" deviceset="RESISTOR" device="_0603" value="6.8k 1%">
-<attribute name="HOUSEPART" value="1"/>
+<attribute name="HOUSEPART" value="0"/>
+<attribute name="MPN" value="RC0603FR-076K8L"/>
 </part>
 <part name="C12" library="mfpassives" deviceset="CAPACITOR_NP" device="_0603" value=".1uF 100V">
-<attribute name="HOUSEPART" value="1"/>
-<attribute name="MPN" value="MF-CAP-0603-0.1uF"/>
+<attribute name="HOUSEPART" value="0"/>
+<attribute name="MPN" value="GRM188R72A104KA35D"/>
 </part>
 <part name="GND7" library="supply1" deviceset="GND" device=""/>
@@
 <part name="R21" library="mfpassives" deviceset="RESISTOR" device="_0603" value="33k">
 <attribute name="HOUSEPART" value="1"/>
+<attribute name="MPN" value="RC0603FR-0733KL"/>
 </part>
 <part name="P+17" library="supply1" deviceset="VCC" device=""/>
@@
 <part name="R24" library="mfpassives" deviceset="RESISTOR" device="_0603" value="0">
 <attribute name="HOUSEPART" value="1"/>
+<attribute name="MPN" value="MF-RES-0603-0"/>
 </part>
 <part name="R25" library="mfpassives" deviceset="RESISTOR" device="_0603" value="DNP">
 <attribute name="HOUSEPART" value="1"/>
+<attribute name="POPULATE" value="0"/>
 </part>
 <part name="C23" library="mfpassives" deviceset="CAPACITOR_NP" device="_0603" value="DNP">
@@
 <part name="R26" library="mfpassives" deviceset="RESISTOR" device="_0603" value="0">
 <attribute name="HOUSEPART" value="1"/>
+<attribute name="MPN" value="MF-RES-0603-0"/>
 </part>
 <part name="D9" library="power_dist" deviceset="SMBJ51CA-E3/52" device="214AB" value="SMBJ51CA-E3/52214AB">
@@
 </part>
 <part name="R3" library="mfpassives" deviceset="RESISTOR" device="_0603" value="200k 1%">
-<attribute name="HOUSEPART" value="1"/>
+<attribute name="HOUSEPART" value="0"/>
+<attribute name="MPN" value="RC0603FR-07200KL"/>
 </part>
 <part name="R16" library="mfpassives" deviceset="RESISTOR" device="_0603" value="100k">
 <attribute name="HOUSEPART" value="1"/>
+<attribute name="MPN" value="MF-RES-0603-100K"/>
 </part>
 <part name="GND15" library="supply1" deviceset="GND" device=""/>
 <part name="R17" library="mfpassives" deviceset="RESISTOR" device="_0603" value="200k 1%">
-<attribute name="HOUSEPART" value="1"/>
+<attribute name="HOUSEPART" value="0"/>
+<attribute name="MPN" value="RC0603FR-07200KL"/>
 </part>
 <part name="GND19" library="supply1" deviceset="GND" device=""/>
@@
 <attribute name="MPN" value="ZXMP10A13FTA"/>
 </part>
-<part name="R18" library="mfpassives" deviceset="RESISTOR" device="_0603" value="100k 1%">
-<attribute name="HOUSEPART" value="1"/>
+<part name="R18" library="mfpassives" deviceset="RESISTOR" device="_0603" value="140k 1%">
+<attribute name="HOUSEPART" value="0"/>
+<attribute name="MPN" value="RC0603FR-07140KL"/>
 </part>
 <part name="R19" library="mfpassives" deviceset="RESISTOR" device="_0603" value="499k 1%">
-<attribute name="HOUSEPART" value="1"/>
+<attribute name="HOUSEPART" value="0"/>
+<attribute name="MPN" value="RC0603FR-07499KL"/>
 </part>
 <part name="GND23" library="supply1" deviceset="GND" device=""/>
 <part name="R20" library="mfpassives" deviceset="RESISTOR" device="_0603" value="47k 1%">
-<attribute name="HOUSEPART" value="1"/>
-</part>
-<part name="R22" library="mfpassives" deviceset="RESISTOR" device="_0603" value="200k 1%">
-<attribute name="HOUSEPART" value="1"/>
+<attribute name="HOUSEPART" value="0"/>
+<attribute name="MPN" value="RC0603FR-0747KL"/>
+</part>
+<part name="R22" library="mfpassives" deviceset="RESISTOR" device="_0603" value="100k">
+<attribute name="HOUSEPART" value="1"/>
+<attribute name="MPN" value="MF-RES-0603-100K"/>
 </part>
 <part name="D6" library="mfdiscretesemi" deviceset="DIODES" device="_SOD-123" technology="_1N4148" value="3V ZENER">
 <attribute name="HOUSEPART" value=""/>
-<attribute name="MPN" value="MMSZ5223BT1G"/>
+<attribute name="MPN" value="MMSZ4682T1G"/>
 <attribute name="URL" value=""/>
 </part>
@@
 <text x="518.16" y="177.8" size="1.778" layer="91">PC13/PA15/PC6 Version
 101</text>
+<text x="-55.88" y="-10.16" size="1.778" layer="91" rot="R180">If this is revved, put a zener in
+parallel with R20 so that R20
+can be equal to R22.</text>
 </plain>
 <instances>
@@
 <attribute name="NAME" x="231.5054" y="31.98206875" size="2.083590625" layer="95" ratio="6" rot="SR0"/>
 <attribute name="VALUE" x="230.8931" y="29.4471" size="2.085490625" layer="96" ratio="6" rot="SR0"/>
+<attribute name="MPN" x="205.74" y="22.86" size="1.778" layer="96" display="off"/>
+<attribute name="POPULATE" x="205.74" y="22.86" size="1.778" layer="96" display="off"/>
 </instance>
 <instance part="GND10" gate="1" x="203.2" y="7.62" smashed="yes">
@@
 <attribute name="NAME" x="-7.62" y="-21.86" size="2.0828" layer="95" ratio="10" rot="SR0"/>
 <attribute name="VALUE" x="-7.62" y="-57.34" size="2.0828" layer="96" ratio="10" rot="SR0"/>
+<attribute name="MPN" x="5.08" y="-38.1" size="1.778" layer="96" display="off"/>
+<attribute name="POPULATE" x="5.08" y="-38.1" size="1.778" layer="96" display="off"/>
 </instance>
 <instance part="R7" gate="G$1" x="43.18" y="-40.64" smashed="yes" rot="R180">
